Commit message: 1.更新了sphere和obb的性能分析脚本 2.一个新的用于分析sphere CHT的脚本

File: data/robots/franka_description/franka_panda.urdf (robot description, URDF)
Before this commit: robot panda, 15 links, 14 joints
Links:
- link base_link: mass None -> 0.01
- link ee_link: mass None -> 0.001
- link panda_hand: mass None -> 0.01
- link panda_leftfinger: mass None -> 0.001
- link panda_link0: mass None -> 0.01
- link panda_link8: mass None -> 0.001
- link panda_rightfinger: mass None -> 0.001

Commit message: 1.修复了collision_env中config加载到robot球体模型和urdf不一致的问题 2.修复了bit_star算法中可能出现的数值错误 3.添加了一下辅助测试程序

File: data/robots/franka_description/franka_panda.urdf (robot description, URDF)
Before this commit: robot panda, 15 links, 14 joints
Joints:
- joint panda_finger_joint1: limit lower=0.0 upper=0.04 effort=20 velocity=0.2 -> (none); origin xyz=0 0 0.0584 rpy=0 0 0 -> xyz=0 0.04 0.0584 rpy=0 0 0; type prismatic -> fixed
- joint panda_finger_joint2: limit lower=0.0 upper=0.04 effort=20 velocity=0.2 -> (none); origin xyz=0 0 0.0584 rpy=0 0 0 -> xyz=0 -0.04 0.0584 rpy=0 0 0; type prismatic -> fixed
