Commit message: add panda urdf to robot model

File: data/robots/iiwa_allegro_description/iiwa.urdf (robot description, URDF)
Before this commit: robot kuka_iiwa, 10 links, 9 joints
Links:
- link iiwa7_link_0: geometry collision mesh filename=meshes/iiwa7/collision/link_0.obj; visual mesh filename=meshes/iiwa7/collision/link_0.obj
- link iiwa7_link_1: geometry collision mesh filename=meshes/iiwa7/collision/link_1.obj; visual mesh filename=meshes/iiwa7/collision/link_1.obj
- link iiwa7_link_2: geometry collision mesh filename=meshes/iiwa7/collision/link_2.obj; visual mesh filename=meshes/iiwa7/collision/link_2.obj
- link iiwa7_link_3: geometry collision mesh filename=meshes/iiwa7/collision/link_3.obj; visual mesh filename=meshes/iiwa7/collision/link_3.obj
- link iiwa7_link_4: geometry collision mesh filename=meshes/iiwa7/collision/link_4.obj; visual mesh filename=meshes/iiwa7/collision/link_4.obj
- link iiwa7_link_5: geometry collision mesh filename=meshes/iiwa7/collision/link_5.obj; visual mesh filename=meshes/iiwa7/collision/link_5.obj
- link iiwa7_link_6: geometry collision mesh filename=meshes/iiwa7/collision/link_6.obj; visual mesh filename=meshes/iiwa7/collision/link_6.obj
- link iiwa7_link_7: geometry collision mesh filename=meshes/iiwa7/collision/link_7.obj; visual mesh filename=meshes/iiwa7/collision/link_7.obj

Commit message: 1.重新调整了pred_trace_generation.py,基于robot_env和sphere_as库进行了重新实现，并更新了相关的命令行参数和错误处理逻辑。 2.调整了robot_env,添加了robot_name和urdf_path参数的对应关系

File: data/robots/iiwa_allegro_description/iiwa.urdf (robot description, URDF)
Before this commit: robot kuka_iiwa, 10 links, 9 joints
Links:
- link base_link: mass None -> 1
- link iiwa7_link_ee: mass None -> 1
